File: evoluent/evoluent.kicad_pcb (KiCad board)
At the start: 2 copper layers, 35 x 54 mm, 30 parts, among them J1 USB_A, J2 Main switches, J3 Thumb switches, J4 Rear lights, J5 Programming header, Q1 2N7002E, U1 ATmega32U4-AU, U2 TLV70019_SOT23-5, U3 PMW3360-T2QU, U4 MCP1700-3302E_SOT23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

Commit message: v0.4
Parts:
- U1: value ATmega32U4-AU -> ATmega32U4-M; footprint Package_QFP:TQFP-44_10x10mm_P0.8mm -> Package_DFN_QFN:QFN-44-1EP_7x7mm_P0.5mm_EP5.2x5.2mm
- Y1: value 8MHz CSTNE8M00G550000R0 -> 16MHz CSTNE16M0V530000R0
- moved Q1 0.55 mm to (139.9, 123.1)
- moved U2 0.11 mm to (153.5, 100.8)
Connections:
- U1 pad 22: Net-(U1-Pad22) -> unconnected-(U1-PD5-Pad22)
- U1 pad 33: Net-(U1-Pad33) -> unconnected-(U1-~{HWB}/PE2-Pad33)
- U1 pad 38: Net-(U1-Pad38) -> unconnected-(U1-PF5-Pad38)
- U1 pad 39: Net-(U1-Pad39) -> unconnected-(U1-PF4-Pad39)
- U1 pad 40: Net-(U1-Pad40) -> unconnected-(U1-PF1-Pad40)
- U1 pad 41: Net-(U1-Pad41) -> unconnected-(U1-PF0-Pad41)
- U1 pad 42: Net-(U1-Pad42) -> unconnected-(U1-AREF-Pad42)
- U1 pad 8: Net-(U1-Pad8) -> unconnected-(U1-PB0-Pad8)
- U2 pad 4: Net-(U2-Pad4) -> unconnected-(U2-NC-Pad4)
- U3 pad 1: Net-(U3-Pad1) -> unconnected-(U3-NC-Pad1)
- U3 pad 14: Net-(U3-Pad14) -> unconnected-(U3-NC-Pad14)
- U3 pad 16: Net-(U3-Pad16) -> unconnected-(U3-NC-Pad16)
- U3 pad 2: Net-(U3-Pad2) -> unconnected-(U3-NC-Pad2)
- U3 pad 6: Net-(U3-Pad6) -> unconnected-(U3-NC-Pad6)
- U3 pad 7: Net-(U3-Pad7) -> unconnected-(U3-NRESET-Pad7)
- U3 pad 9: Net-(U3-Pad9) -> unconnected-(U3-MOTION-Pad9)
Routing:
- net GND: track 48.8 -> 60.0 mm, vias 19 -> 18
- net +3V3: track 97.8 -> 104.8 mm, vias 3 -> 7
- net +5V: track 141.0 -> 136.3 mm
- net /M_LED2: track 26.4 -> 29.4 mm
- net /LED_ON: track 8.29 -> 11.2 mm
- net /M_LED1: track 14.6 -> 17.4 mm
- net /M_THUMB_BOTTOM: track 19.6 -> 22.4 mm
- net /M_UNK2: track 38.0 -> 40.7 mm
- net /M_LED0: track 12.8 -> 15.5 mm
- net Net-(U1-D+): track 3.05 -> 5.73 mm
- net /M_3: track 47.0 -> 49.7 mm
- net Net-(U1-D-): track 5.14 -> 7.75 mm
- net /M_UNK1: track 42.9 -> 45.4 mm
- net /FILT_SCROLL_A: track 31.2 -> 33.7 mm
- net /CS: track 25.7 -> 28.2 mm
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Other:
- net class Default removed
- rule pad_to_mask_clearance: 0.051 -> 0.038
- board text added: "Evoluent VMC/D PMW3360 board v0.4 mon.im 2023"
- board text removed: "Evoluent VMC/D PMW3360 board v0.3 mon.im 2020"
